File: ESP12+mosfet+1117.brd (EAGLE design)
At the start: 59.4 x 45.7 mm, 36 parts, among them IC1 LM1117T-3.3-V, Q1 IRLZ34N, Q2 IRLZ34N, Q3 IRLZ34N, Q4 IRLZ34N

Commit message: New version
Parts:
- added C4: 100nF, rcl:C0805
- added C5: 10uF, resistor:E2-4
- LED1: device led:LED5MM -> led:LED3MM
- moved R10 2.56 mm to (19.4, 17.8)
- turned IC1 to 180 degrees
Connections:
- net +12V: now also C4.1
- net +3V3: now also C5.+, JP2.2, JP2.4, JP2.6, JP4.1, JP4.3, JP4.5; no longer JP4.2, JP4.4, JP4.6
- net GND: now also C4.2, C5.-, JP4.2, JP4.4, JP4.6; no longer JP2.2, JP2.4, JP2.6, JP4.1, JP4.3, JP4.5
Routing:
- net +3V3: track 86.0 -> 80.1 mm
- net +12V: track 87.2 -> 91.4 mm
- net GPIO16: track 38.1 -> 41.0 mm
- net N$1: track 3.18 -> 4.54 mm
Other:
- board text added: "ESP-12 LED driver v1.0"
- board text added: "Q1-Q4: IRLZ34N IC1: LD1117V33"
- board text added: "R1-R9: 10k R10: 150R C1-C4: 100n C5: 10u"
- board text removed: "ESP-12 LED driver"
- board text removed: "R1-R9: 10k R10: 150R C1-C3: 100n Q1-Q4: IRLZ34N IC1: LD1117V33"
